File: missionpcb_kicad/projects/ECG20/MissionPCB.kicad_pcb (KiCad board)
At the start: 2 copper layers, 72 x 38 mm, 20 parts, among them J1 BM02B-SRSS-TB, J2 JST SH 3 pin, J3 JST SH 4 pin, U1 MSP430FR2433, U2 ADS1292R [APPROX], U3 MDBT42Q-512KV2, U4 TPS62740 [APPROX], U5 MCP73831

Commit message: Build engineering review timeline, wearable budgets and native CAD assembly
Parts:
- moved J1 32.0 mm to (138.0, 119.0), turned to -90 degrees
- moved U2 17.1 mm to (125.0, 125.0)
- moved R3 15.0 mm to (143.3, 120.2)
- moved C6 13.5 mm to (143.3, 118.7)
- moved C7 10.7 mm to (130.3, 122.2)
- moved C3 10.3 mm to (119.8, 118.2)
- moved R2 9.27 mm to (128.3, 118.2)
- moved C2 9.23 mm to (127.8, 119.7)
- moved L1 9.17 mm to (136.2, 108.3)
- moved C1 8.93 mm to (140.3, 125.7)
- moved U4 8.56 mm to (139.5, 110.0)
- moved R1 7.70 mm to (130.3, 119.2), turned to -90 degrees
- moved U3 7.62 mm to (109.0, 113.0), turned to 0 degrees
- moved C5 7.32 mm to (137.8, 115.7), turned to -90 degrees
- moved U5 6.41 mm to (148.9, 119.0)
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Other:
- board text added: "J1 WATCH"
- board text added: "J2 WATCH"
- board text added: "J3 WATCH"
- board text added: "U1 ERROR"
- board text added: "U2 ERROR"
- board text added: "[MPCB] J1 REVIEW [2]"
- board text added: "[MPCB] J2 REVIEW [2]"
- board text added: "[MPCB] J3 REVIEW [2]"
- board text added: "[MPCB] U1 FAIL [1]"
- board text added: "[MPCB] U2 FAIL [1]"
- board text removed: "[MPCB AREA] C3 ERROR"
- board text removed: "[MPCB AREA] J1 WATCH"
- board text removed: "[MPCB AREA] J2 WATCH"
- board text removed: "[MPCB AREA] J3 WATCH"
- board text removed: "[MPCB AREA] L1 ERROR"
- board text removed: "[MPCB AREA] U1 ERROR"
- board text removed: "[MPCB AREA] U2 ERROR"
- board text removed: "[MPCB AREA] U3 ERROR"
- board text removed: "[MPCB AREA] U4 ERROR"
- board text removed: "[MPCB AREA] U5 ERROR"
- board text removed: "[MPCB] C3 FAIL [1]"
- board text removed: "[MPCB] J1 REVIEW [8]"
- board text removed: "[MPCB] J2 REVIEW [8]"
- board text removed: "[MPCB] J3 REVIEW [8]"
- board text removed: "[MPCB] L1 FAIL [1,4]"
- board text removed: "[MPCB] U1 FAIL [2]"
- board text removed: "[MPCB] U2 FAIL [2,3,4,5,7]"
- board text removed: "[MPCB] U3 FAIL [6]"
- board text removed: "[MPCB] U4 FAIL [3,6,7]"
- board text removed: "[MPCB] U5 FAIL [5]"
